File: pcb/KR1801.kicad_sch (KiCad schematic)
At the start: 1 part

Commit message: ECB
Parts:
- added J1: ECB, Connector_DIN:DIN41612_R_3x32_Male_Horizontal_THT, symbol ECB:ECB_RB-6
- gave numbers to parts that had none: 1
Connections:
- net CLC: now reaches U1.1 (CLC)
- net CLC: now also J1.c29 (CLC)
- net ~{SACK}: now reaches U1.2 (~{SACK})
- net GND: now reaches U1.21 (GND)
- net GND: now also J1.a32 (GND), J1.b32 (GND), J1.c32 (GND)
- net ~{BEN}: now reaches U1.28 (~{BSY})
- net ~{DCLO}: now reaches U1.29 (~{DCLO})
- net ~{DCLO}: now also J1.c31 (~{RESET})
- net ~{ACLO}: now reaches U1.30 (~{ACLO})
- net ~{ACLO}: now also J1.c20 (~{NMI})
- net ~{IRQ1}: now reaches U1.31 (~{IRQ1})
- net ~{IRQ1}: now also J1.c25 (~{HALT})
- net ~{INIT}: now reaches U1.34 (~{INIT})
- net ~{INIT}: now also J1.c26 (~{RESOUT})
- net ~{VIRQ}: now reaches U1.35 (VIRQ)
- net ~{VIRQ}: now also J1.c21 (~{INT})
- net ~{IAKO}: now reaches U1.36 (IAKO)
- net ~{IAKO}: now also J1.b25 (~{INTA})
- net ~{DOUT}: now reaches U1.37 (~{DOUT})
- net ~{DOUT}: now also J1.c22 (~{WR})
- net ~{DIN}: now reaches U1.38 (~{DIN})
- net ~{DIN}: now also J1.c24 (~{RD})
- net ~{RPLY}: now reaches U1.39 (~{RPLY})
- net ~{RPLY}: now also J1.a22 (~{RDY})
- net ~{DMGO}: now reaches U1.4 (~{DMGO})
- net ~{DMGO}: now also J1.a31 (~{BUSAK})
- net ~{WTBT}: now reaches U1.40 (~{WTBT})
- net ~{ALE}: now reaches U1.41 (~{SYNC})
- net VCC: now reaches U1.42 (VCC)
- net VCC: now also J1.a1 (VCC), J1.b1 (VCC), J1.c1 (VCC)
- net ~{DMR}: now reaches U1.5 (~{DMR})
- net ~{DMR}: now also J1.a11 (~{BUSRQ})
Other:
- note added: "Latch address on falling edge"
- note added: "NOT"

Commit message: 3D models
Parts:
- added R1, R2, R3, R4, R5, R6, R7: R, symbol Device:R
Connections:
- net VCC: now also R1.2, R2.2, R3.2, R4.2, R5.2, R6.2, R7.2
- net ~{DMR}: now also R5.1
- net ~{IRQ1}: now also R1.1
- net ~{RPLY}: now also R7.1
- net ~{SACK}: now also R6.1
- net ~{VIRQ}: now also R4.1
- net ~{IRQ2}: now reaches U1.32 (IRQ2)
- net ~{IRQ2}: now also R2.1
- net ~{IRQ3}: now reaches U1.33 (IRQ3)
- net ~{IRQ3}: now also R3.1
Other:
- moved on the sheet: J1, U1

Commit message: more docs and boot
Parts:
- added R10, R11, R9: 0R, symbol Device:R
- added R12, R13, R14, R15: R, symbol Device:R
- added R8: OR, symbol Device:R
Connections:
- net ~{BEN} is gone; now on net AB.OE: U1.28 (~{PA1})
- net VCC: now also R10.2, R11.2, R12.2, R13.2, R14.2, R15.2, R8.2, R9.2
- net ~{ACLO}: no longer J1.c20 (~{NMI})
- net at U1.27 (~{PA0}): now also R8.1
- net AB.OE: now reaches U1.28 (~{PA1})
- net AB.OE: now also R15.1
- net at U1.3 (~{DMGI}): now also R10.1
- net at U1.6 (~{SP}): now also R11.1
- net ~{SEL1}: now reaches U1.7 (~{SEL1})
- net ~{SEL1}: now also R13.1
- net ~{SEL2}: now reaches U1.8 (~{SEL2})
- net ~{SEL2}: now also R14.1
- new net: R9.1, U1.28 (~{PA1})
- new net ~{NMI}: J1.c20 (~{NMI}), R12.1
Other:
- note added: "50Hz timer sync falling edge on raising edge of CLC"
- note added: "Release ~{INIT} to high after ~{DCLO} is high"
- note added: "sync falling edge on raising edge of CLC"

Commit message: random placement test
Parts:
- added U2, U3: 74LS573, Package_SO:SOIC-20W_7.5x12.8mm_P1.27mm, symbol 74xx:74LS573
- added U4, U5: 74LS245, Package_SO:SOIC-20W_7.5x12.8mm_P1.27mm, symbol 74xx:74LS245
- R1, R10, R11, R12, R13, R14, R15, R2, R3, R4, R5, R6, R7, R9: footprint (none) -> Resistor_SMD:R_0603_1608Metric_Pad0.98x0.95mm_HandSolder
- R8: value OR -> 0R; footprint (none) -> Resistor_SMD:R_0603_1608Metric_Pad0.98x0.95mm_HandSolder
Connections:
- net ~{INIT} is gone; now on net ~{DCLO}: J1.c26 (~{RESOUT}), U1.34 (~{INIT})
- net GND: now also U4.10 (GND), U5.10 (GND)
- net VCC: now also U4.20 (VCC), U5.20 (VCC)
- net AD1: now reaches U1.10 (~{AD1})
- net AD1: now also U2.3 (D1), U4.3 (A1)
- net AD2: now reaches U1.11 (~{AD2})
- net AD2: now also U2.4 (D2), U4.4 (A2)
- net AD3: now reaches U1.12 (~{AD3})
- net AD3: now also U2.5 (D3), U4.5 (A3)
- net AD4: now reaches U1.13 (~{AD4})
- net AD4: now also U2.6 (D4), U4.6 (A4)
- net AD5: now reaches U1.14 (~{AD5})
- net AD5: now also U2.7 (D5), U4.7 (A5)
- net AD6: now reaches U1.15 (~{AD6})
- net AD6: now also U2.8 (D6), U4.8 (A6)
- net AD7: now reaches U1.16 (~{AD7})
- net AD7: now also U2.9 (D7), U4.9 (A7)
- net AD8: now reaches U1.17 (~{AD8})
- net AD8: now also U3.2 (D0), U5.2 (A0)
- net AD9: now reaches U1.18 (~{AD9})
- net AD9: now also U3.3 (D1), U5.3 (A1)
- net AD10: now reaches U1.19 (~{AD10})
- net AD10: now also U3.4 (D2), U5.4 (A2)
- net AD11: now reaches U1.20 (~{AD11})
- net AD11: now also U3.5 (D3), U5.5 (A3)
- net AD12: now reaches U1.22 (~{AD12})
- net AD12: now also U3.6 (D4), U5.6 (A4)
- net AD13: now reaches U1.23 (~{AD13})
- net AD13: now also U3.7 (D5), U5.7 (A5)
- net AD14: now reaches U1.24 (~{AD14})
- net AD14: now also U3.8 (D6), U5.8 (A6)
- net AD15: now reaches U1.25 (~{AD15})
- net AD15: now also U3.9 (D7), U5.9 (A7)
- net at R9.1: now also U1.26 (~{PA1}); no longer U1.28 (~{PA1})
- net AD0: now reaches U1.9 (~{AD0})
- net AD0: now also U2.2 (D0), U4.2 (A0)
- net A14: now reaches J1.a18 (A14)
- net A14: now also U3.13 (Q6)
- net DB5: now reaches J1.a2 (D5)
- net DB5: now also U4.13 (B5)
- net A13: now reaches J1.a29 (A13)
- net A13: now also U3.14 (Q5)
- net DB6: now reaches J1.a3 (D6)
- net DB6: now also U4.12 (B6)
- net A9: now reaches J1.a30 (A9)
- net A9: now also U3.18 (Q1)
- net DB3: now reaches J1.a4 (D3)
- net DB3: now also U4.15 (B3)
- net DB4: now reaches J1.a5 (D4)
- net DB4: now also U4.14 (B4)
- net A2: now reaches J1.a6 (A2)
- net A2: now also U2.17 (Q2)
- net A4: now reaches J1.a7 (A4)
- net A4: now also U2.15 (Q4)
- net A5: now reaches J1.a8 (A5)
- net A5: now also U2.14 (Q5)
- net A6: now reaches J1.a9 (A6)
- net A6: now also U2.13 (Q6)
- net DB12: now reaches J1.b10 (D12)
- net DB12: now also U5.14 (B4)
- net DB13: now reaches J1.b11 (D13)
- net DB13: now also U5.13 (B5)
- net DB14: now reaches J1.b12 (D14)
- net DB14: now also U5.12 (B6)
- net DB15: now reaches J1.b13 (D15)
- net DB15: now also U5.11 (B7)
- net DB8: now reaches J1.b6 (D8)
- net DB8: now also U5.18 (B0)
- net DB9: now reaches J1.b7 (D9)
- net DB9: now also U5.17 (B1)
- net DB10: now reaches J1.b8 (D10)
- net DB10: now also U5.16 (B2)
- net DB11: now reaches J1.b9 (D11)
- net DB11: now also U5.15 (B3)
- net DB1: now reaches J1.c14 (D1)
- net DB1: now also U4.17 (B1)
- net A11: now reaches J1.c17 (A11)
- net A11: now also U3.16 (Q3)
- net A10: now reaches J1.c18 (A10)
- net A10: now also U3.17 (Q2)
- net DB0: now reaches J1.c2 (D0)
- net DB0: now also U4.18 (B0)
- net A12: now reaches J1.c27 (A12)
- net A12: now also U3.15 (Q4)
- net A15: now reaches J1.c28 (A15)
- net A15: now also U3.12 (Q7)
- net DB7: now reaches J1.c3 (D7)
- net DB7: now also U4.11 (B7)
- net DB2: now reaches J1.c4 (D2)
- net DB2: now also U4.16 (B2)
- net A0: now reaches J1.c5 (A0)
- net A0: now also U2.19 (Q0)
- net A3: now reaches J1.c6 (A3)
- net A3: now also U2.16 (Q3)
- net A1: now reaches J1.c7 (A1)
- net A1: now also U2.18 (Q1)
- net A8: now reaches J1.c8 (A8)
- net A8: now also U3.19 (Q0)
- net A7: now reaches J1.c9 (A7)
- net A7: now also U2.12 (Q7)

Commit message: most of the glue logic and controls
Parts:
- removed R1, R14, R2, R3, R6: R, Resistor_SMD:R_0603_1608Metric_Pad0.98x0.95mm_HandSolder, symbol Device:R
- removed U2, U3: 74LS573, Package_SO:SOIC-20W_7.5x12.8mm_P1.27mm, symbol 74xx:74LS573
- removed U4, U5: 74LS245, Package_SO:SOIC-20W_7.5x12.8mm_P1.27mm, symbol 74xx:74LS245
- added R18: 0R, Resistor_SMD:R_0603_1608Metric_Pad0.98x0.95mm_HandSolder, symbol Device:R
- R11: value 0R -> R
- R15: value R -> WEAKR; footprint Resistor_SMD:R_0603_1608Metric_Pad0.98x0.95mm_HandSolder -> esistor_SMD:R_0603_1608Metric_Pad0.98x0.95mm_HandSolder
Connections:
- net ~{DCLO}: no longer J1.c26 (~{RESOUT}), J1.c31 (~{RESET}), U1.34 (~{INIT})
- net ~{DMR}: now also R12.1; no longer R5.1
- net ~{DS1}: now also J1.b29 (~{DS1})
- net ~{IRQ1}: no longer J1.c25 (~{HALT})
- net ~{NMI}: no longer R12.1
- net ~{RPLY}: no longer J1.a22 (~{RDY}), R7.1
- net ~{SACK}: now also R13.1
- net ~{SEL1}: now also R4.1; no longer R13.1
- net ~{SEL2}: now also R5.1
- net ~{VIRQ}: no longer R4.1
- net ~{SP}: now reaches U1.6 (~{SP})
- net ~{SP}: no longer R11.1
- net at J1.b28 (~{DS0}): now also R18.1
- net AB.OE renamed ~{BSY}
- net ~{BSY}: now also R7.1; no longer R15.1
- net ~{ALE} renamed ~{SYNC}
- net ~{SYNC}: now also R11.1, R18.2
- new net ~{HALT}: J1.c25 (~{HALT})
- new net ~{INIT}: J1.c26 (~{RESOUT}), R15.1, U1.34 (~{INIT})
- new net ~{RDY}: J1.a22 (~{RDY})
- new net ~{RESET}: J1.c31 (~{RESET})
Other:
- added sheet glue (glue.kicad_sch)
- note added: "Processor"
- note removed: "50Hz timer sync falling edge on raising edge of CLC"
- note removed: "Latch address on falling edge"
- note removed: "NOT"
- note removed: "sync falling edge on raising edge of CLC"

Commit message: final logic, gal, 3D
Parts:
- J1: footprint Connector_DIN:DIN41612_R_3x32_Male_Horizontal_THT -> Connector_DIN:DIN41612_C_3x32_Male_Horizontal_THT
Changed lines of the file:
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@@
       (effects (font (size 1.27 1.27)))
     )
-    (property "Footprint" "Connector_DIN:DIN41612_R_3x32_Male_Horizontal_THT" (at 40.64 17.78 0)
+    (property "Footprint" "Connector_DIN:DIN41612_C_3x32_Male_Horizontal_THT" (at 40.64 17.78 0)
       (effects (font (size 1.27 1.27)) hide)
     )

Commit message: /init
Parts:
- added R50: 0R, Resistor_SMD:R_0603_1608Metric_Pad0.98x0.95mm_HandSolder, symbol Device:R
- R18: now not fitted; now left out of the parts list
Connections:
- net ~{DS1}: now also R50.2; no longer J1.b29 (~{DS1})
- new net: J1.b29 (~{DS1}), R50.1
Other:
- note removed: "Release ~{INIT} to high after ~{DCLO} is high"
Changed lines of the file:
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@@
   (junction (at 36.83 119.38) (diameter 0) (color 0 0 0 0)
-  )
-  (junction (at 255.27 157.48) (diameter 0) (color 0 0 0 0)
-  )
-  (wire (pts (xy 255.27 160.02) (xy 255.27 157.48))
-    (stroke (width 0) (type default))
-  )
-  (wire (pts (xy 255.27 157.48) (xy 256.54 157.48))
-    (stroke (width 0) (type default))
   )
   (wire (pts (xy 177.8 149.86) (xy 180.34 149.86))
@@
     (stroke (width 0) (type default))
   )
-  (wire (pts (xy 256.54 160.02) (xy 255.27 160.02))
-    (stroke (width 0) (type default))
-  )
   (wire (pts (xy 39.37 119.38) (xy 41.91 119.38))
     (stroke (width 0) (type default))
   )
   (wire (pts (xy 177.8 154.94) (xy 180.34 154.94))
-    (stroke (width 0) (type default))
-  )
-  (wire (pts (xy 251.46 157.48) (xy 255.27 157.48))
     (stroke (width 0) (type default))
   )
@@
     (fill (type none))
   )
-  (text "Release ~{INIT} to high after ~{DCLO} is high" (at 243.84 165.1 0)
-    (effects (font (size 1.27 1.27)) (justify left bottom))
-  )
   (text "Processor" (at 142.24 24.13 0)
     (effects (font (size 1.27 1.27)) (justify left bottom))
@@
     )
   )
-  (global_label "~{INIT}" (shape output) (at 256.54 160.02 0) (fields_autoplaced)
-    (effects (font (size 1.27 1.27)) (justify left))
-    (property "Intersheetrefs" "${INTERSHEET_REFS}" (at 263.0329 160.02 0)
-      (effects (font (size 1.27 1.27)) (justify left) hide)
-    )
-  )
   (global_label "DB3" (shape bidirectional) (at 26.67 40.64 180) (fields_autoplaced)
     (effects (font (size 1.27 1.27)) (justify right))
@@
     )
   )
-  (global_label "~{DS1}" (shape input) (at 26.67 76.2 180) (fields_autoplaced)
-    (effects (font (size 1.27 1.27)) (justify right))
-    (property "Intersheetrefs" "${INTERSHEET_REFS}" (at 19.9958 76.2 0)
+  (global_label "~{DS1}" (shape input) (at 19.05 76.2 180) (fields_autoplaced)
+    (effects (font (size 1.27 1.27)) (justify right))
+    (property "Intersheetrefs" "${INTERSHEET_REFS}" (at 12.3758 76.2 0)
       (effects (font (size 1.27 1.27)) (justify right) hide)
     )
@@
   )
   (symbol (lib_id "Device:R") (at 22.86 73.66 270) (unit 1)
-    (in_bom yes) (on_board yes) (dnp no)
+    (in_bom no) (on_board yes) (dnp yes)
     (property "Reference" "R18" (at 22.86 73.66 90)
       (effects (font (size 1.27 1.27)))
@@
         )
       )
+    )
+  )
+  (symbol (lib_id "Device:R") (at 22.86 76.2 270) (unit 1)
+    (in_bom no) (on_board yes) (dnp yes)
+    (property "Reference" "R50" (at 22.86 76.2 90)
+      (effects (font (size 1.27 1.27)))
+    )
+    (property "Value" "0R" (at 22.86 72.39 90)
+      (effects (font (size 1.27 1.27)) hide)
+    )
+    (property "Footprint" "Resistor_SMD:R_0603_1608Metric_Pad0.98x0.95mm_HandSolder" (at 22.86 74.422 90)
+      (effects (font (size 1.27 1.27)) hide)
+    )
+    (property "Datasheet" "~" (at 22.86 76.2 0)
+      (effects (font (size 1.27 1.27)) hide)
+    )
+    (pin "1")
+    (pin "2")
+    (instances
+      (project "KR1801"
+        (path "/68e08f4a-84cb-4510-afcb-23087110769d"
+          (reference "R50") (unit 1)
+        )
+      )

Commit message: full? schematics
Parts:
- J1: value ECB -> Eurocard UNIBUS
Changed lines of the file:
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@@
   )
   (symbol (lib_id "ECB:ECB_RB-6") (at 39.37 12.7 0) (unit 1)
-    (in_bom yes) (on_board yes) (dnp no) (fields_autoplaced)
+    (in_bom yes) (on_board yes) (dnp no)
     (property "Reference" "J1" (at 39.37 33.02 0) (do_not_autoplace)
       (effects (font (size 1.27 1.27)))
     )
-    (property "Value" "ECB" (at 39.37 35.56 0) (do_not_autoplace)
+    (property "Value" "Eurocard UNIBUS" (at 39.37 43.18 90) (do_not_autoplace)
       (effects (font (size 1.27 1.27)))
     )
