File: pcb/KR1801.kicad_pcb (KiCad board)
At the start: 2 copper layers, 160 x 100 mm, 51 parts, among them J1 Eurocard UNIBUS, SW1 Reset Vector, SW2 Opts, SW3 NMI, SW4 RESET, U1 К1801ВМ1, U10 GAL16V8, U2 74HC564, U3 74HC564, U4 74HC640, U5 74HC640, U6 74AHC273, U7 74LS240, U8 74LS240, U9 74LS259

Commit message: placement/routing
Parts:
- added R1: 0R, Resistor_SMD:R_0603_1608Metric_Pad0.98x0.95mm_HandSolder, F.Cu at (195.0, 134.8)
- added R10: 0R, Resistor_SMD:R_0603_1608Metric_Pad0.98x0.95mm_HandSolder, F.Cu at (154.5, 71.5)
- added R11: R, Resistor_SMD:R_0603_1608Metric_Pad0.98x0.95mm_HandSolder, F.Cu at (155.4, 114.1)
- added R12: R, Resistor_SMD:R_0603_1608Metric_Pad0.98x0.95mm_HandSolder, F.Cu at (152.0, 70.1)
- added R13: R, Resistor_SMD:R_0603_1608Metric_Pad0.98x0.95mm_HandSolder, F.Cu at (157.3, 70.2)
- added R14: R, Resistor_SMD:R_0603_1608Metric_Pad0.98x0.95mm_HandSolder, F.Cu at (169.1, 131.4)
- added R16: 0R, Resistor_SMD:R_0603_1608Metric_Pad0.98x0.95mm_HandSolder, F.Cu at (169.1, 133.2)
- added R17: 0R, Resistor_SMD:R_0603_1608Metric_Pad0.98x0.95mm_HandSolder, F.Cu at (169.2, 135.6)
- added R18: 0R, Resistor_SMD:R_0603_1608Metric_Pad0.98x0.95mm_HandSolder, F.Cu at (132.1, 121.1)
- added R2: 0R, Resistor_SMD:R_0603_1608Metric_Pad0.98x0.95mm_HandSolder, F.Cu at (192.4, 127.6)
- added R3: R, Resistor_SMD:R_0603_1608Metric_Pad0.98x0.95mm_HandSolder, F.Cu at (193.9, 131.6)
- added R35: RLED, Resistor_SMD:R_0603_1608Metric_Pad0.98x0.95mm_HandSolder, F.Cu at (68.5, 122.9)
- added R4: R, Resistor_SMD:R_0603_1608Metric_Pad0.98x0.95mm_HandSolder, F.Cu at (149.7, 70.2)
- added R45: R, Resistor_SMD:R_0603_1608Metric_Pad0.98x0.95mm_HandSolder, F.Cu at (169.1, 129.3)
- added R46: RLED, Resistor_SMD:R_0603_1608Metric_Pad0.98x0.95mm_HandSolder, F.Cu at (64.6, 145.6)
- added R47: 0R, Resistor_SMD:R_0603_1608Metric_Pad0.98x0.95mm_HandSolder, F.Cu at (160.0, 116.2)
- added R48: WEAKR, Resistor_SMD:R_0603_1608Metric_Pad0.98x0.95mm_HandSolder, F.Cu at (146.6, 113.6)
- added R5: R, Resistor_SMD:R_0603_1608Metric_Pad0.98x0.95mm_HandSolder, F.Cu at (148.2, 70.1)
- added R50: 0R, Resistor_SMD:R_0603_1608Metric_Pad0.98x0.95mm_HandSolder, F.Cu at (190.1, 140.5)
- added R6: 0R, Resistor_SMD:R_0603_1608Metric_Pad0.98x0.95mm_HandSolder, F.Cu at (169.1, 127.5)
- added R7: R, Resistor_SMD:R_0603_1608Metric_Pad0.98x0.95mm_HandSolder, F.Cu at (138.4, 115.0)
- added R8: 0R, Resistor_SMD:R_0603_1608Metric_Pad0.98x0.95mm_HandSolder, F.Cu at (136.1, 115.0)
- added R9: 0R, Resistor_SMD:R_0603_1608Metric_Pad0.98x0.95mm_HandSolder, F.Cu at (134.4, 115.1)
- added U11: MCP100-475D, Package_TO_SOT_SMD:SOT-23-3, F.Cu at (120.3, 121.7)
- moved R44 36.1 mm to (166.4, 60.2), turned to 180 degrees
- moved X1 31.6 mm to (166.4, 65.9), turned to 180 degrees
- moved U10 18.7 mm to (143.7, 124.4)
- moved U1 15.1 mm to (157.0, 80.8)
Connections:
- U3 pad 13: A14 -> A12
- U3 pad 14: A13 -> A14
- U3 pad 15: A12 -> A13
- U3 pad 6: AD12 -> AD13
- U3 pad 7: AD13 -> AD14
- U3 pad 8: AD14 -> AD12
Routing:
- net AD12: track 0.00 -> 81.9 mm, vias 0 -> 2
- net AD11: track 0.00 -> 81.5 mm
- net AD9: track 0.00 -> 77.9 mm
- net AD10: track 0.00 -> 77.2 mm
- net AD14: track 0.00 -> 75.8 mm
- net AD13: track 0.00 -> 74.5 mm
- net AD8: track 0.00 -> 73.5 mm
- net AD15: track 0.00 -> 72.5 mm
- net DB1: track 0.00 -> 72.3 mm, vias 0 -> 2
- net A8: track 0.00 -> 51.2 mm, vias 0 -> 2
- net AD7: track 25.7 -> 72.9 mm
- net ~{DMR}: track 0.00 -> 47.0 mm, vias 0 -> 2
- net AD5: track 25.6 -> 70.6 mm
- net AD6: track 25.7 -> 69.3 mm
- net AD3: track 25.7 -> 68.4 mm
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- added copper zone on B.Cu, net GND
- added copper zone on F.Cu, net GND
